Commit message: Clean workspace, fixed URDF and removed extra TF sources

File: valet_parking_amr/my_robot_description/urdf/common_properties.xacro (robot description, xacro)
@@ -1,62 +1,36 @@
 <?xml version="1.0"?>
 <robot xmlns:xacro="http://www.ros.org/wiki/xacro">
-  <!-- ===================== -->
-  <!-- Common Materials      -->
-  <!-- ===================== -->
-  <xacro:macro name="common_materials">
-    <material name="green">
-      <color rgba="0 1 0 1"/>
+    <material name="blue">
+        <color rgba="0 0 0.5 1" />
     </material>
     <material name="grey">
-      <color rgba="0.5 0.5 0.5 1"/>
+        <color rgba="0.5 0.5 0.5 1" />
     </material>
-  </xacro:macro>
-  <!-- ===================== -->
-  <!-- Box Inertia           -->
-  <!-- ===================== -->
-  <xacro:macro name="box_inertia" params="m x y z o_xyz o_rpy">
-    <inertial>
-      <mass value="${m}"/>
-      <origin xyz="${o_xyz}" rpy="${o_rpy}"/>
-      <inertia
-        ixx="${m/12.0 * (z*z + y*y)}"
-        ixy="0"
-        ixz="0"
-        iyy="${m/12.0 * (x*x + z*z)}"
-        iyz="0"
-        izz="${m/12.0 * (x*x + y*y)}"/>
-    </inertial>
-  </xacro:macro>
-  <!-- ===================== -->
-  <!-- Cylinder Inertia      -->
-  <!-- ===================== -->
-  <xacro:macro name="cylinder_inertia" params="m r l o_xyz o_rpy">
-    <inertial>
-      <mass value="${m}"/>
-      <origin xyz="${o_xyz}" rpy="${o_rpy}"/>
-      <inertia
-        ixx="${m/12.0 * (3*r*r + l*l)}"
-        ixy="0"
-        ixz="0"
-        iyy="${m/12.0 * (3*r*r + l*l)}"
-        iyz="0"
-        izz="${m/2.0 * (r*r)}"/>
-    </inertial>
-  </xacro:macro>
-  <!-- ===================== -->
-  <!-- Sphere Inertia        -->
-  <!-- ===================== -->
-  <xacro:macro name="sphere_inertia" params="m r o_xyz o_rpy">
-    <inertial>
-      <mass value="${m}"/>
-      <origin xyz="${o_xyz}" rpy="${o_rpy}"/>
-      <inertia
-        ixx="${2.0/5.0 * m * r * r}"
-        ixy="0"
-        ixz="0"
-        iyy="${2.0/5.0 * m * r * r}"
-        iyz="0"
-        izz="${2.0/5.0 * m * r * r}"/>
-    </inertial>
-  </xacro:macro>
+    <xacro:macro name="box_inertia" params="m x y z o_xyz o_rpy">
+        <inertial>
+            <mass value="${m}" />
+            <origin xyz="${o_xyz}" rpy="${o_rpy}" />
+            <inertia ixx="${(m/12) * (y*y + z*z)}" ixy="0" ixz="0"
+                     iyy="${(m/12) * (x*x + z*z)}" iyz="0"
+                     izz="${(m/12) * (x*x + y*y)}" />
+        </inertial>
+    </xacro:macro>
+    <xacro:macro name="cylinder_inertia" params="m r l o_xyz o_rpy">
+        <inertial>
+            <mass value="${m}" />
+            <origin xyz="${o_xyz}" rpy="${o_rpy}" />
+            <inertia ixx="${(m/12) * (3*r*r + l*l)}" ixy="0" ixz="0"
+                     iyy="${(m/12) * (3*r*r + l*l)}" iyz="0"
+                     izz="${(m/2) * (r*r)}" />
+        </inertial>
+    </xacro:macro>
+    <xacro:macro name="sphere_inertia" params="m r o_xyz o_rpy">
+        <inertial>
+            <mass value="${m}" />
+            <origin xyz="${o_xyz}" rpy="${o_rpy}" />
+            <inertia ixx="${(2/5) * m * r * r}" ixy="0" ixz="0"
+                     iyy="${(2/5) * m * r * r}" iyz="0"
+                     izz="${(2/5) * m * r * r}" />
+        </inertial>
+    </xacro:macro>
 </robot>

File: valet_parking_amr/my_robot_description/urdf/mobile_base_gazebo.xacro (robot description, xacro)
@@ -1,36 +1,27 @@
 <?xml version="1.0"?>
 <robot xmlns:xacro="http://www.ros.org/wiki/xacro">
-  <!-- ===================== -->
-  <!-- Caster Wheel Friction -->
-  <!-- ===================== -->
-  <gazebo reference="caster_wheel_link">
-    <mu1 value="0.1"/>
-    <mu2 value="0.1"/>
-  </gazebo>
-  <!-- ===================== -->
-  <!-- Diff Drive Plugin     -->
-  <!-- ===================== -->
-  <gazebo>
-    <plugin
-      filename="gz-sim-diff-drive-system"
-      name="gz::sim::systems::DiffDrive">
-      <left_joint>base_left_wheel_joint</left_joint>
-      <right_joint>base_right_wheel_joint</right_joint>
-      <wheel_separation>0.45</wheel_separation>
-      <wheel_radius>0.1</wheel_radius>
-      <frame_id>odom</frame_id>
-      <child_frame_id>base_footprint</child_frame_id>
-    </plugin>
-  </gazebo>
-  <!-- ===================== -->
-  <!-- Joint State Publisher -->
-  <!-- ===================== -->
-  <gazebo>
-    <plugin
-      filename="gz-sim-joint-state-publisher-system"
-      name="gz::sim::systems::JointStatePublisher">
-      <joint_name>base_left_wheel_joint</joint_name>
-      <joint_name>base_right_wheel_joint</joint_name>
-    </plugin>
-  </gazebo>
+    <gazebo reference="caster_wheel_link">
+        <mu1 value="0.1" />
+        <mu2 value="0.1" />
+    </gazebo>
+    <gazebo>
+        <plugin
+            filename="gz-sim-diff-drive-system"
+            name="gz::sim::systems::DiffDrive">
+            <left_joint>base_left_wheel_joint</left_joint>
+            <right_joint>base_right_wheel_joint</right_joint>
+            <wheel_separation>0.45</wheel_separation>
+            <wheel_radius>0.1</wheel_radius>
+            <frame_id>odom</frame_id>
+            <child_frame_id>base_footprint</child_frame_id>
+        </plugin>
+    </gazebo>
+    <gazebo>
+        <plugin
+            filename="gz-sim-joint-state-publisher-system"
+            name="gz::sim::systems::JointStatePublisher">
+            <joint_name>base_left_wheel_joint</joint_name>
+            <joint_name>base_right_wheel_joint</joint_name>
+        </plugin>
+    </gazebo>
 </robot>

File: valet_parking_amr/my_robot_description/urdf/my_robot.urdf.xacro (robot description, xacro)
@@ -1,8 +1,7 @@
 <?xml version="1.0"?>
 <robot name="my_robot" xmlns:xacro="http://www.ros.org/wiki/xacro">
-  <xacro:include filename="common_properties.xacro"/>
-  <xacro:common_materials/>
-  <xacro:include filename="mobile_base.xacro"/>
-  <xacro:include filename="mobile_base_gazebo.xacro"/>
-  <xacro:include filename="camera.xacro"/>
+    <xacro:include filename="common_properties.xacro" />
+    <xacro:include filename="mobile_base.xacro" />
+    <xacro:include filename="mobile_base_gazebo.xacro" />
+    <xacro:include filename="camera.xacro" />
 </robot>
